Commit message: updated amcl launch file
Signed-off-by: Ekanshh <fictious.ekansh@gmail.com>

File: my_robot/urdf/robby.xacro (robot description, xacro)
@@ -151,5 +151,5 @@
     <visual name='visual'>
       <geometry>
-        <mesh filename= "package://pkg_1/meshes/hokuyo.dae" />
+        <mesh filename= "package://my_robot/meshes/hokuyo.dae" />
       </geometry>
     </visual>
